File: Phase_1/PCB Circuit/Module/module_phase1.sch (EAGLE design)
At the start: 1 part, among them U1 MSP430G2553IN20

Commit message: Circuits + Gearbox
Parts:
- added LED1: (no value), microbuilder:LED0805
- added R1, R2: (no value), microbuilder:RESISTOR0805
- added U2: 74LVX4245MTCX, 74LVX4245MTCX:74LVX4245MTCX
Connections:
- new net /RST: R2.1, U1.!RST!/NMI/SBWTDIO
- new net 5.0V: U2.VCCA
- new net A1: U1.P2.2/TA1.1, U2.B0
- new net A1O: U2.A0
- new net A2: U1.P2.0/TA1.0, U2.B1
- new net A2O: U2.A1
- new net B1: U1.P2.4/TA1.2, U2.B3
- new net B1O: U2.A3
- new net B2: U1.P2.3/TA1.0, U2.B4
- new net B2O: U2.A4
- new net CS: U1.P1.5/TA0.0/UCB0CLK/UCA0STE/A5/CA5/TMS
- new net LED: LED1.A, U1.P1.7/A7/CA7/CAOUT/UCB0SIMO/UCB0SDA/TDO/TDI
- new net N$1: LED1.C, R1.1
- new net PWMA: U1.P2.1/TA1.1, U2.B2
- new net PWMAO: U2.A2
- new net PWMB: U1.P2.5/TA1.2, U2.B5
- new net PWMBO: U2.A5
- new net SCLK: U1.P1.4/SMCLK/UCB0STE/UCA0CLK/A4/VREF/PVEREF/PCA4/TCK
- new net SENSORA: U1.P1.3/ADC10CLK/A3/VREF/NVEREF/NCA3I/CAOUT
- new net SENSORB: U1.P1.6/TA0.1/A6/CA6/UCB0SOMI/UCB0SCL/TDI/TCLK
- new net SIMO: U1.P1.2/TA0.1/UCA0TXD/UCA0SIMO/A2/CA2
- new net SOMI: U1.P1.1/TA0.0/UCA0RXD/UCA0SOMI/A1/CA1
- new net STATE_SEL: U1.P1.0/TA0CLK/ACLK/A0/CA0
- net 3.3V: now also R2.2, U2.VCCB, U2.VCCB_2
- net GND: now also R1.2, U2.GND, U2.GND_2, U2.GND_3, U2.T/~R, U2.~OE

Commit message: GEARBOX Finished with stl
Parts:
- added C1: (no value), microbuilder:CAP_CERAMIC0805
- added C2: (no value), microbuilder:CAP_ELECTROLYTICPANASONIC_C
Connections:
- net 3.3V: now also C1.P$1, C2.+
- net GND: now also C1.P$2, C2.-
Changed lines of the file:
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@@
 <part name="U$8" library="microbuilder" deviceset="GND" device=""/>
 <part name="U$9" library="microbuilder" deviceset="5.0V" device=""/>
+<part name="C1" library="microbuilder" deviceset="CAP_CERAMIC" device="0805"/>
+<part name="C2" library="microbuilder" deviceset="CAP_ELECTROLYTIC" device="PANASONIC_C"/>
 </parts>
 <sheets>
@@
 <attribute name="VALUE" x="56.896" y="36.576" size="1.27" layer="96"/>
 </instance>
+<instance part="C1" gate="G$1" x="147.32" y="68.58" smashed="yes">
+<attribute name="NAME" x="149.86" y="71.12" size="1.27" layer="95" font="vector"/>
+<attribute name="VALUE" x="149.86" y="68.58" size="1.27" layer="96" font="vector"/>
+</instance>
+<instance part="C2" gate="G$1" x="154.94" y="68.58" smashed="yes">
+<attribute name="NAME" x="157.48" y="71.12" size="1.27" layer="95" font="vector"/>
+<attribute name="VALUE" x="157.48" y="68.58" size="1.27" layer="96" font="vector"/>
+</instance>
 </instances>
 <busses>
@@
 <wire x1="127" y1="83.82" x2="129.54" y2="83.82" width="0.1524" layer="91"/>
 <wire x1="129.54" y1="83.82" x2="129.54" y2="86.36" width="0.1524" layer="91"/>
+<wire x1="129.54" y1="83.82" x2="147.32" y2="83.82" width="0.1524" layer="91"/>
+<pinref part="C1" gate="G$1" pin="P$1"/>
+<wire x1="147.32" y1="83.82" x2="147.32" y2="73.66" width="0.1524" layer="91"/>
+<pinref part="C2" gate="G$1" pin="+"/>
+<wire x1="147.32" y1="73.66" x2="154.94" y2="73.66" width="0.1524" layer="91"/>
 </segment>
 <segment>
@@
 <pinref part="U$2" gate="G$1" pin="GND"/>
 <wire x1="127" y1="48.26" x2="127" y2="45.72" width="0.1524" layer="91"/>
+<pinref part="C1" gate="G$1" pin="P$2"/>
+<pinref part="C2" gate="G$1" pin="-"/>
+<wire x1="147.32" y1="66.04" x2="152.4" y2="66.04" width="0.1524" layer="91"/>
+<wire x1="152.4" y1="66.04" x2="154.94" y2="66.04" width="0.1524" layer="91"/>
+<wire x1="152.4" y1="66.04" x2="152.4" y2="48.26" width="0.1524" layer="91"/>
+<wire x1="152.4" y1="48.26" x2="127" y2="48.26" width="0.1524" layer="91"/>
 </segment>
 <segment>
