File: Phase_2/PCB Circuit/TX_test.sch (EAGLE design)
At the start: 3 parts

Commit message: PCB
Parts:
- added LED1: (no value), Phase_2:LED3MM
- added R1: (no value), Phase_2:R-US_0204/7
- added U$4: MSP430G2553IN20, Phase_2:MSP430G2553IN20
Connections:
- new net CS: U$4.P$7
- new net INT: U$1.P$14, U$4.P$5
- new net N$10: LED1.C, R1.2
- new net N$5: U$1.P$7, U$2.P$10
- new net N$6: U$1.P$3, U$2.P$6
- new net N$7: U$1.P$4, U$2.P$7
- new net N$8: U$1.P$6, U$2.P$8
- new net N$9: U$1.P$5, U$2.P$11
- new net PORT0: U$1.P$8, U$4.P$8
- new net PORT1: U$1.P$9, U$4.P$9
- new net PORT2: U$1.P$10, U$4.P$10
- new net PORT3: U$1.P$11, U$4.P$11
- new net PORT4: U$1.P$12, U$4.P$12
- new net PORT5: U$1.P$13, U$4.P$13
- new net PORT6: U$1.P$19, U$4.P$19
- new net PORT7: U$1.P$18, U$4.P$18
- new net SCLK: U$4.P$6
- new net SIMO: U$4.P$4
- new net SOMI: U$4.P$3
- new net SS: LED1.A, U$1.P$2, U$4.P$2
- new net SW: U$1.P$15
- new net X: U$4.P$15
- new net Y: U$4.P$14
- net N$1: now also U$1.P$16, U$4.P$1, U$4.P$16
- net N$3: now also R1.1, U$4.P$20
Other:
- note added: "Auto Sender"
- note added: "RF"
- note added: "RF_TX_uC"
