File: Phase_2/PCB Circuit/TX/test/TX_test.brd (EAGLE design)
At the start: 90.2 x 58.1 mm, 9 parts

Commit message: 5+4
Parts:
- moved LED1 6.40 mm to (63.3, 42.0)
- moved R1 6.40 mm to (72.2, 40.7)
- moved U$1 6.40 mm to (44.3, 25.5)
- moved U$2 6.40 mm to (17.6, 26.8)
- moved U$3 6.40 mm to (2.35, 40.7)
- moved U$4 6.40 mm to (63.3, 25.5)
- moved U$5 6.40 mm to (41.7, 47.1)
- moved U$6 6.40 mm to (53.1, 3.89)
- moved U$7 6.40 mm to (77.3, 19.1)
Other:
- board size 90.2 x 58.1 mm -> 80.2 x 53.1 mm
