File: Phase_2/PCB Circuit/TX/test/TX_test.sch (EAGLE design)
At the start: 9 parts

Commit message: 5+4
Changed lines of the file:
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@@
 <wire x1="121.92" y1="38.1" x2="121.92" y2="10.16" width="0.1524" layer="91"/>
 <junction x="55.88" y="38.1"/>
+<label x="-15.24" y="40.64" size="1.778" layer="95"/>
 </segment>
 </net>
